File: DC5V_DC5V3V3.kicad_pcb (KiCad board)
At the start: 2 copper layers, 21.5 x 19.2 mm, 24 parts, among them J1 Vout1, J2 Vout2, Q1 BSS138, U1 LM1117-3.3

Commit message: Сформирован перечень элементов, 3D-модель, исправлены ошибки, реализована панелизация платы.
Parts:
- J1: footprint Modules:PinHeader_1x04_P2.54mm_Horizontal -> Modules:PinHeader_1x04_P2.54mm_Horizontal_short
- J2: footprint Modules:PinHeader_1x03_P2.54mm_Horizontal -> Modules:PinHeader_1x03_P2.54mm_Horizontal_short
