File: DC5V_DC5V3V3.sch (KiCad schematic (older format))
At the start: 27 parts, among them J1 Vout1, J2 Vout2, Q1 BSS138, U1 LM1117-3.3

Commit message: Окончена трассировка печатной платы
Parts:
- removed JP1: 5V_en, Jumper:SolderJumper-2_P1.3mm_Open_TrianglePad1.0x1.5mm, symbol Jumper:SolderJumper_2_Open
- removed JP2: 5VL_en, Jumper:SolderJumper-2_P1.3mm_Open_TrianglePad1.0x1.5mm, symbol Jumper:SolderJumper_2_Open
- removed JP3: N_en, Jumper:SolderJumper-2_P1.3mm_Open_TrianglePad1.0x1.5mm, symbol Jumper:SolderJumper_2_Open
- removed JP4: 3V3_en, Jumper:SolderJumper-2_P1.3mm_Open_TrianglePad1.0x1.5mm, symbol Jumper:SolderJumper_2_Open
- added C12: 470uF, Capacitor_Tantalum_SMD:CP_EIA-7343-15_Kemet-W, symbol Device:CP_Small
- J1: footprint Connector_PinHeader_2.54mm:PinHeader_1x04_P2.54mm_Horizontal -> Modules:PinHeader_1x04_P2.54mm_Horizontal
- J2: footprint Connector_PinHeader_2.54mm:PinHeader_1x03_P2.54mm_Horizontal -> Modules:PinHeader_1x03_P2.54mm_Horizontal
- renumbered C9 to C10, C12 to C13, C13 to C14, C14 to C15, C15 to C16, C10 to C8, C8 to C9
Connections:
- net +5P0 is gone; now on net +5P: C5.2, C6.2, D1.3 (~CE), D1.6 (VOUT), Q1.1 (G), R1.1, R2.2
- net +3.3VP: now also C15.2, C16.2, U1.2 (VO)
- net +5VP: now also C10.2, C9.2, PS1.4 (+Vout), C12.1
- net GND2: now also C10.1, C9.1, PS1.3 (-Vout), C12.2
Other:
- moved on the sheet: C1, C11, C13, C14, C15, C16, C3, C5, C6, C7, C8, D1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

Commit message: Сформирован перечень элементов, 3D-модель, исправлены ошибки, реализована панелизация платы.
Parts:
- J1: footprint Modules:PinHeader_1x04_P2.54mm_Horizontal -> Modules:PinHeader_1x04_P2.54mm_Horizontal_short
- J2: footprint Modules:PinHeader_1x03_P2.54mm_Horizontal -> Modules:PinHeader_1x03_P2.54mm_Horizontal_short
Changed lines of the file:
@@
 F 0 "J2" H 6050 1725 50  0000 C CNN
 F 1 "Vout2" H 6025 1325 50  0000 C CNN
-F 2 "Modules:PinHeader_1x03_P2.54mm_Horizontal" H 6050 1525 50  0001 C CNN
+F 2 "Modules:PinHeader_1x03_P2.54mm_Horizontal_short" H 6050 1525 50  0001 C CNN
 F 3 "~" H 6050 1525 50  0001 C CNN
 	1    6050 1525
@@
 F 0 "J1" H 5175 1725 50  0000 C CNN
 F 1 "Vout1" H 5175 1225 50  0000 C CNN
-F 2 "Modules:PinHeader_1x04_P2.54mm_Horizontal" H 5175 1525 50  0001 C CNN
+F 2 "Modules:PinHeader_1x04_P2.54mm_Horizontal_short" H 5175 1525 50  0001 C CNN
 F 3 "~" H 5175 1525 50  0001 C CNN
 	1    5175 1525
